File: eagle/Pico Audio v0.13.sch (EAGLE design)
At the start: 62 parts, among them IC1 MIC_I2S_SPH0645, J1 OUTL, J2 OUTR, J3 TinyPICO, J4 TinyPICO, J5 SPI Breakout, J6 PicoAudio, U1 MAX98306ETD+T, U2 UDA1334ATS, X1 STEREOJACKSTX3120-5B

Commit message: v0.13 Update
Parts:
- removed LOGO2: OSHW-LOGOM, SparkFun-Aesthetics:OSHW-LOGOM
- removed U$12, U$13, U$14: MOUNTINGHOLE2.5, microbuilder:MOUNTINGHOLE2.5
- added C19: 0.1uF, rcl:C-USC0402K
- added C20, C21: 1uF, rcl:C-USC0402K
- added J8: Pin Out 1, SparkFun-Connectors:CONN_08NO_SILK_FEMALE_PTH
- added LOGO1: OSHW-LOGOM, SparkFun-Aesthetics:OSHW-LOGOM
- added MH1, MH2, MH3: MOUNTINGHOLE2.5, microbuilder:MOUNTINGHOLE2.5
- added R21: 4.7K, rcl:R-US_R0402
- added R22: 270, rcl:R-US_R0402
- added S6: MOMENTARY-SWITCH-SPST-SMD-4.6X2.8MM, SparkFun-Switches:MOMENTARY-SWITCH-SPST-SMD-4.6X2.8MM
- added U3: PCF8574, AK74:PCF8574
- added U4: NCP170AMX300TCG, NCP170AMX300TCG:NCP170AMX300TCG
- AK74LOGO2: value AK74_LOGO -> AK74_LOGOAK74_LOGO_SMALL; device AK74:AK74_LOGO -> AK74:AK74_LOGOAK74_LOGO_SMALL
- C10, C11: value 0.1uF -> 10uF; device rcl:C-USC0402K -> rcl:C-USC0603K
- C12: value 10uF -> 0.1uF; device rcl:C-USC0603K -> rcl:C-USC0402K
- C16: value 220pf -> 1uF
- C3: value 1uF -> 10uF; device rcl:C-USC0402K -> rcl:C-USC0603K
- C4: value 1uF -> 0.1uF
- C5: value 10uF -> 1uF; device rcl:C-USC0603K -> rcl:C-USC0402K
- C6: value 0.1uF -> 220pf
- C7: value 10uF -> 47uF; device rcl:C-USC0603K -> rcl:C-USC1210K
- C9: value 47uF -> 0.1uF; device rcl:C-USC1210K -> rcl:C-USC0402K
- J1: value OUTL -> OUTR
- J2: value OUTR -> OUTL
- J3: value TinyPICO -> GPIO Expander Pins; device UnexpectedMaker:TINYPICO_HEADER_10NO_SILK_PTH_FEMALE -> SparkFun-Connectors:CONN_08NO_SILK_FEMALE_PTH
- J5: value SPI Breakout -> TinyPICO; device SparkFun-Connectors:CONN_05NO_SILK -> UnexpectedMaker:TINYPICO_HEADER_10NO_SILK_PTH_FEMALE
- J6: value PicoAudio -> Pin Out 2; device SparkFun-Connectors:CONN_041X04_NO_SILK -> SparkFun-Connectors:CONN_07NO_SILK
- R10, R11: value 10K -> 100
- R13: value 68 -> 10K
- R14: value 10K -> 270
- R16: value 10K -> 100K
- R17: value 270 -> 100K
- R18, R19: value 100K -> 10K
- R20: value 270 -> 4.7K
- R8: value 100 -> 68
- R9: value 100 -> 10K
- U1: value MAX98306ETD+T -> UDA1334ATS; device microbuilder:AUDIOAMP_MAX98306 -> microbuilder:AUDIO_I2S_UDA1334""
- U2: value UDA1334ATS -> MAX98306ETD+T; device microbuilder:AUDIO_I2S_UDA1334"" -> microbuilder:AUDIOAMP_MAX98306
Connections:
- removed net GPIO14: IC1.BCLK, J3.6
- removed net GPIO15: J3.7, R13.1
- removed net GPIO18: J4.3, J5.4, SD1.SCK, SDCRD.A
- removed net GPIO19: J4.2, J5.3, R15.2, SD1.MISO
- removed net GPIO22: J4.5, U2.DATAI
- removed net GPIO23: J4.1, J5.2, R14.2, SD1.MOSI
- removed net GPIO25: J3.10, J5.5
- removed net GPIO26: J3.9, U2.WS
- removed net GPIO32: J4.7, S2.1
- removed net GPIO33: J4.8, S1.1
- removed net GPIO4: IC1.WS, J3.5
- removed net GPIO5: J4.4, R16.1, R17.1, SD1.!CS
- removed net N$6: R4.2, U2.MUTE
- new net +3V3#2: C1.1, C19.1, C2.1, C21.1, FB2.2, R20.2, R21.2, U1.VDDD, U3.VCC, U4.OUT
- new net DAC_BCK: J4.9, U1.BCK
- new net DAC_DIN: J5.5, U1.DATAI
- new net DAC_WS: J4.10, U1.WS
- new net MIC_BCK: IC1.BCLK, J4.6, J8.7
- new net MIC_DOUT: J4.7, J8.5, R8.1
- new net MIC_WS: IC1.WS, J4.5, J8.6
- new net MISO: J5.2, J6.2, R12.2, SD1.MISO
- new net MOSI: J5.1, J6.1, R9.2, SD1.MOSI
- new net MUTE: J8.8, R4.2, U1.MUTE
- new net P0: J3.1, U3.P0
- new net P1: J3.2, U3.P1
- new net P2: J3.3, U3.P2
- new net P3: J3.4, U3.P3
- new net P4: J3.5, U3.P4
- new net P5: J3.6, S1.1, U3.P5
- new net P6: J3.7, S2.1, U3.P6
- new net P7: J3.8, S3.1, U3.P7
- new net SCK: J5.3, J6.3, SD1.SCK, SDCRD.A
- new net SCL: J5.8, J6.7, R20.1, U3.SCL
- new net SDA: J5.7, J6.6, R21.1, U3.SDA
- new net SD_CS: J5.4, R13.1, R14.1, SD1.!CS
- net +3V3: now also C12.1, C5.1, C6.1, J4.4, J8.1, R13.2; no longer C1.1, C15.1, C16.1, C17.1, C18.1, C2.1, C7.1, FB2.2, J3.4, J6.2, JP1.3, R1.1, R16.2, R19.2, U1.PVDD@1, U1.PVDD@2, U2.VDDD
- net +5V: now also C17.1, C18.1, C20.1, J4.3, J8.2, JP1.3, R15.1, R17.2, U2.PVDD@1, U2.PVDD@2, U4.EN, U4.IN; no longer J3.3, J6.1
- net AGND: now also C3.2, C4.2, C9.2, R18.1, R19.1, U1.VSSA, U2.INL-, U2.INR-; no longer C12.2, C5.2, C6.2, R10.1, R12.1, U1.INL-, U1.INR-, U2.VSSA
- net DEEM: now also J8.4, U1.DEEM/CLKOUT; no longer J6.3, U2.DEEM/CLKOUT
- net GAIN1: now also U2.GAIN; no longer U1.GAIN
- net GND: now also C12.2, C19.2, C20.2, C21.2, C5.2, C6.2, J4.2, J5.10, J8.3, R1.1, R12.1, R16.1, R22.1, R9.1, S6.2, U1.VSSD, U2.PGND@1, U2.PGND@2, U2.THERMAL, U3.A0, U3.A1, U3.A2, U3.GND, U4.EXP, U4.GND; no longer C15.2, C16.2, C7.2, J3.2, J4.10, J6.4, R11.1, R14.1, R15.1, R18.1, R20.1, U1.PGND@1, U1.PGND@2, U1.THERMAL, U2.VSSD
- net GPIO21: now also J5.6, J6.4; no longer J4.6, J5.1
- net GPIO27: now also J4.8, J6.5; no longer J3.8, U2.BCK
- net N$1: now also C3.1, C4.1, U1.VDDA; no longer C5.1, C6.1, U2.VDDA
- net N$10: now also U1.PLL0; no longer U2.PLL0
- net N$11: now also U1.SYSCLK/PLL1; no longer U2.SYSCLK/PLL1
- net N$14: now also C9.1, U1.VREF(DAC); no longer C12.1, U2.VREF(DAC)
- net N$15: now also C7.1, U1.VOUTL; no longer C8.1, U2.VOUTL
- net N$16: now also C8.2, R11.2; no longer C9.2, R9.2
- net N$17: now also J2.2, U2.OUTR-; no longer J1.2, U1.OUTR-
- net N$18: now also J1.2, U2.OUTL-; no longer J2.2, U1.OUTL-
- net N$19: now also C7.2, R10.2; no longer C8.2, R8.2
- net N$2: now also C15.1, U2.INL+; no longer C3.1, U1.INL+
- net N$20: now also R2.2; no longer R11.2
- net N$21: now also C8.1, U1.VOUTR; no longer C9.1, U2.VOUTR
- net N$22: now also R8.2; no longer R13.2
- net N$24: now also R17.1; no longer R19.1
- net N$25: now also R16.2; no longer R18.2
- net N$26: now also J1.1, U2.OUTL+; no longer J2.1, U1.OUTL+
- net N$27: now also R14.2; no longer R17.2
- net N$28: now also J2.1, U2.OUTR+; no longer J1.1, U1.OUTR+
- net N$3: now also R1.2, U1.SFOR1; no longer R2.2, U2.SFOR1
- net N$4: now also C16.1, U2.INR+; no longer C4.1, U1.INR+
- net N$5: now also U1.SFOR0; no longer U2.SFOR0
- net N$8: now also R22.2; no longer R20.2
- net RESET: now also J5.9, S6.1; no longer J4.9, S3.1
- net SHUTDOWN: now also R15.2, U2.SHDN; no longer R1.2, U1.SHDN
- net VBAT: now also J4.1; no longer J3.1
- net VINL: now also C15.2, R18.2; no longer C3.2, R10.2
- net VINR: now also C16.2, R19.2; no longer C4.2, R12.2
- net VOUTL: now also R10.1; no longer R8.1
- net VOUTR: now also R11.1; no longer R9.1
Other:
- note added: "+3V3"
- note added: "+5V"
- note added: "GND"
- note added: "GPIO14"
- note added: "GPIO15"
- note added: "GPIO18"
- note added: "GPIO19"
- note added: "GPIO21"
- note added: "GPIO22"
- note added: "GPIO23"
- note added: "GPIO25"
- note added: "GPIO26"
- note added: "GPIO27"
- note added: "GPIO32"
- note added: "GPIO33"
- note added: "GPIO4"
- note added: "GPIO5"
- note added: "NCP167BMX330TBG"
- note added: "POWER"
- note added: "RESET"
- note added: "SCL"
- note added: "SDA"
- note added: "TinyPICO Header"
- note added: "VBAT"
- moved on the sheet: C1, C10, C11, C12, C13, C14, C15, C16, C17, C18, C2, C3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
