File: eagle/Pico Audio v0.13.brd (EAGLE design)
At the start: 32.8 x 56.9 mm, 93 parts, among them IC1 MIC_I2S_SPH0645, J1 TinyPICO, J2 TinyPICO, J3 Pin Out 1, J4 GPIO Expander Pins, J5 OUTR, J6 OUTL, J7 Pin Out 2, U1 UDA1334ATS, U2 TPA6132A2RTER, U3 NCP170AMX300TCG, U4 NC7SZ04, U5 MAX98306ETD+T, U6 PCF8574, X1 STEREOJACKSTX3120-5B

Commit message: Revert "Board Update"
This reverts commit 64f88ad06b88c25f0d87ce8718a64f2d2cec739c.
Parts:
- removed AK74LOGO1: AK74_LOGOAK74_LOGO_SMALL, AK74:AK74_LOGO_MEDIUM
- removed C22, C23, C24, C25, C26, C27, C28: 1uF, rcl:C0402K
- removed C29, C31: 0.1uF, rcl:C0402K
- removed C30: 10uF, rcl:C0603K
- removed J7: Pin Out 2, SparkFun-Connectors:1X07_NO_SILK
- removed JP2: SPKGAIN, pinhead:2X04
- removed R23: 100K, rcl:R0402
- removed R24: 10K, rcl:R0402
- removed R25, R26: 270, rcl:R0402
- removed R27, R28: 4.7K, rcl:R0402
- removed S4, S5: SKSCLDE010, AK74:SKSCLDE010
- removed U5: MAX98306ETD+T, microbuilder:TDFN14_3X3MM
- removed U6: PCF8574, AK74:QFN-16-3MM
- added AK74LOGO2: AK74_LOGOAK74_LOGO_SMALL, AK74:AK74_LOGO_MEDIUM
- added J8: Pin Out 1, SparkFun-Connectors:1X08_NO_SILK
- C11: value 0.1uF -> 10uF; device rcl:C0402K -> rcl:C0603K
- C12: value 10uF -> 0.1uF; device rcl:C0603K -> rcl:C0402K
- C15, C5: value 10uF -> 1uF; device rcl:C0603K -> rcl:C0402K
- C16: value 2.2uF -> 1uF
- C17, C3: value 1uF -> 10uF; device rcl:C0402K -> rcl:C0603K
- C18: value 1uF -> 0.1uF
- C19: value 2.2uF -> 0.1uF
- C4: value 220pf -> 0.1uF
- C6: value 0.1uF -> 220pf
- J1: value TinyPICO -> OUTR; device UnexpectedMaker:1X10_NO_SILK -> microbuilder:TERMBLOCK_1X2-3.5MM
- J2: value TinyPICO -> OUTL; device UnexpectedMaker:1X10_NO_SILK -> microbuilder:TERMBLOCK_1X2-3.5MM
- J3: value Pin Out 1 -> GPIO Expander Pins
- J4: value GPIO Expander Pins -> TinyPICO; device SparkFun-Connectors:1X08_NO_SILK -> UnexpectedMaker:1X10_NO_SILK
- J5: value OUTR -> TinyPICO; device microbuilder:TERMBLOCK_1X2-3.5MM -> UnexpectedMaker:1X10_NO_SILK
- J6: value OUTL -> Pin Out 2; device microbuilder:TERMBLOCK_1X2-3.5MM -> SparkFun-Connectors:1X07_NO_SILK
- JP1: value HPGAIN -> GAIN; device pinhead:2X02 -> pinhead:2X04
- R10: value 10K -> 100
- R11: value 220K -> 100
- R12: value 220K -> 10K
- R13: value 100 -> 10K
- R14: value 100 -> 270
- R16: value 270 -> 100K
- R17: value 10K -> 100K
- R19: value 100K -> 10K
- R20: value 49.9K -> 4.7K
- R21: value 270 -> 4.7K
- R22: value 100K -> 270
- R6: value 68 -> 10K
- R8: value 10K -> 68
- S1, S2, S3: value SKSCLDE010 -> MOMENTARY-SWITCH-SPST-SMD-4.6X2.8MM; device AK74:SKSCLDE010 -> SparkFun-Switches:TACTILE_SWITCH_SMD_4.6X2.8MM
- U2: value TPA6132A2RTER -> MAX98306ETD+T; device TPA6132A2RTER:QFN50P300X300X80-16N -> microbuilder:TDFN14_3X3MM
- U3: value NCP170AMX300TCG -> PCF8574; device NCP170AMX300TCG:VREG_NCP170AMX300TCG -> AK74:QFN-16-3MM
- U4: value NC7SZ04 -> NCP170AMX300TCG; device AK74:MICROPAK-6 -> NCP170AMX300TCG:VREG_NCP170AMX300TCG
- moved MH3 51.6 mm to (2.54, 2.06)
- moved MH2 49.1 mm to (2.54, 51.1)
- moved JP1 48.5 mm to (10.3, 2.22), turned to 180 degrees
- moved R17 32.2 mm to (11.1, 8.57), turned to 0 degrees
- moved R14 25.7 mm to (28.6, 17.5), turned to 180 degrees
- moved R21 24.7 mm to (9.37, 37.5), turned to 90 degrees
- moved R22 24.4 mm to (28.6, 22.5), turned to 180 degrees
- moved R20 23.8 mm to (8.10, 37.5), turned to 90 degrees
- moved J4 22.6 mm to (1.37, 32.7), turned to 0 degrees
- moved R16 22.3 mm to (8.57, 8.57), turned to 0 degrees
- moved J5 21.4 mm to (1.37, 17.4), turned to 0 degrees
- moved C12 21.4 mm to (14.9, 10.2)
- moved U4 20.4 mm to (11.0, 37.5), turned to 180 degrees
- moved C10 20.1 mm to (7.30, 30.2)
- moved J3 18.0 mm to (19.2, 46.7), turned to 180 degrees
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- renumbered LED1 to SDCRD, LED2 to PWR
Connections:
- removed net /JACKSENSE: R24.2, U4.4, U5.P$2
- removed net G0: JP1.2, U2.6
- removed net G1: JP1.4, U2.7
- removed net JACKSENSE: C24.1, R20.2, U4.2
- removed net N$12: C18.2, U2.4
- removed net N$13: R17.1, U2.13
- removed net N$23: C19.1, U2.12
- removed net N$29: R18.1, U2.5, X1.2
- removed net N$30: U2.16, X1.5
- removed net N$31: C21.2, U2.11
- removed net N$32: C21.1, U2.9
- removed net N$33: C22.1, U2.8
- removed net N$34: R19.2, R20.1, X1.3
- removed net N$6: C26.1, U5.P$4
- removed net N$7: C28.1, U5.P$6
- removed net N$9: C17.2, U2.1
- new net SHUTDOWN: R15.2, U2.P$2
- new net VINL: C15.2, R18.2, X1.4
- new net VINR: C16.2, R19.2, X1.3
- net +3V3: now also C12.1, C5.1, C6.1, J4.4, J8.1, R13.2; no longer C10.1, C3.1, C4.1, J1.4, J3.1, R15.2
- net +3V3#2: now also C19.1, C21.1, R20.2, R21.2, U4.1; no longer C15.1, C16.1, C23.1, C29.1, JP1.1, JP1.3, R17.2, R19.1, R27.2, R28.2, U2.14, U4.6, U6.1
- net +5V: now also C17.1, C18.1, J4.3, J8.2, JP1.3, R15.1, R17.2, U2.P$11, U2.P$12, U4.3, U4.4; no longer C30.1, C31.1, J1.3, J3.2, JP2.3, R23.2, U3.3, U3.4, U5.P$11, U5.P$12
- net AGND: now also C10.2, C3.2, C4.2, R18.1, R19.1, U2.P$4, U2.P$6; no longer C12.2, C26.2, C28.2, C5.2, C6.2, R11.2, R12.2, R25.1, R26.1, U2.15
- net DAC_BCK: now also J4.9; no longer J1.9
- net DAC_DIN: now also J5.5; no longer J2.5
- net DAC_WS: now also J4.10; no longer J1.10
- net DEEM: now also J8.4; no longer J3.4
- net GAIN1: now also JP1.2, JP1.4, JP1.6, JP1.8, U2.P$5; no longer JP2.2, JP2.4, JP2.6, JP2.8, U5.P$5
- net GND: now also C12.2, C17.2, C18.2, C21.2, C5.2, C6.2, J4.2, J5.10, J8.3, JP1.7, R12.1, R16.1, R6.1, U2.P$1, U2.P$8, U2.P$THERMAL, U3.3, U3.4, U3.9, U3.P$1, U4.2, U4.5; no longer C10.2, C15.2, C16.2, C22.2, C23.2, C24.2, C29.2, C3.2, C30.2, C31.2, C4.2, J1.2, J2.10, J3.3, JP2.7, R10.1, R18.2, R21.1, R24.1, R8.1, S4.3, S4.4, S5.3, S5.4, U2.10, U2.17, U2.2, U2.3, U3.5, U4.3, U5.P$1, U5.P$8, U5.P$THERMAL, U6.2, U6.3, U6.4, U6.9, U6.P$1
- net GPIO21: now also J5.6, J6.4; no longer J2.6, J7.4
- net GPIO27: now also J4.8, J6.5; no longer J1.8, J7.5
- net MIC_BCK: now also J4.6, J8.7; no longer J1.6, J3.7
- net MIC_DOUT: now also J4.7, J8.5, R8.1; no longer J1.7, J3.5, R6.1
- net MIC_WS: now also J4.5, J8.6; no longer J1.5, J3.6
- net MISO: now also J5.2, J6.2, R12.2; no longer J2.2, J7.2, R10.2
- net MOSI: now also J5.1, J6.1; no longer J2.1, J7.1
- net MUTE: now also J8.8; no longer J3.8
- net N$1: now also C3.1, C4.1; no longer C5.1, C6.1
- net N$10: now also R6.2; no longer R7.2
- net N$11: now also R7.2; no longer R8.2
- net N$14: now also C10.1; no longer C12.1
- net N$16: now also R11.2; no longer R12.1, R14.2
- net N$17: now also J2.2, U2.P$9; no longer J6.2, U5.P$9
- net N$18: now also J1.2, U2.P$14; no longer J5.2, U5.P$14
- net N$19: now also R10.2; no longer R11.1, R13.2
- net N$2: now also C15.1, U2.P$3; no longer C25.1, U5.P$3
- net N$20: now also R2.2; no longer R1.2
- net N$22: now also R8.2; no longer R6.2
- net N$24: now also JP1.1, R17.1; no longer JP2.1, R23.1
- net N$25: now also JP1.5, R16.2; no longer JP2.5, R22.2
- net N$26: now also J1.1, U2.P$13; no longer J5.1, U5.P$13
- net N$27: now also R14.2; no longer R16.2
- net N$28: now also J2.1, U2.P$10; no longer J6.1, U5.P$10
- net N$3: now also R1.2; no longer R2.2
- net N$4: now also C16.1, U2.P$7; no longer C27.1, U5.P$7
- net N$8: now also R22.2; no longer R21.2
- net P0: now also J3.1, U3.5; no longer J4.1, U6.5
- net P1: now also J3.2, U3.6; no longer J4.2, U6.6
- net P2: now also J3.3, U3.7; no longer J4.3, U6.7
- net P3: now also J3.4, U3.8; no longer J4.4, S1.1, S1.2, U6.8
- net P4: now also J3.5, U3.10; no longer J4.5, S2.1, S2.2, U6.10
- net P5: now also J3.6, S1.1, S1.2, U3.11; no longer J4.6, S3.1, S3.2, U6.11
- net P6: now also J3.7, S2.1, S2.2, U3.12; no longer J4.7, S4.1, S4.2, U6.12
- net P7: now also J3.8, S3.1, S3.2, U3.13; no longer J4.8, S5.1, S5.2, U6.13
- net RESET: now also J5.9; no longer J2.9
- net SCK: now also J5.3, J6.3; no longer J2.3, J7.3
- net SCL: now also J5.8, J6.7, R20.1, U3.15; no longer J2.8, J7.7, R27.1, U6.15
- net SDA: now also J5.7, J6.6, R21.1, U3.16; no longer J2.7, J7.6, R28.1, U6.16
- net SD_CS: now also J5.4, R13.1, R14.1; no longer J2.4, R15.1, R16.1
- net VBAT: now also J4.1; no longer J1.1
- net VOUTL: now also R10.1, X1.5; no longer C17.1, C25.2, R13.1, R26.2
- net VOUTR: now also R11.1, X1.2; no longer C18.1, C27.2, R14.1, R25.2
Routing:
- net +5V: track 85.1 -> 10.4 mm, vias 3 -> 4
- net P3: track 39.7 -> 6.75 mm
- net GND: track 81.1 -> 54.7 mm, vias 34 -> 28
- net G0: track 26.2 -> 0.00 mm, vias 1 -> 0
- net P4: track 30.6 -> 6.51 mm
- net G1: track 23.9 -> 0.00 mm, vias 1 -> 0
- net N$30: track 23.7 -> 0.00 mm
- net VINL: track 0.00 -> 22.7 mm
- net +3V3#2: track 38.9 -> 16.2 mm, vias 10 -> 6
- net VINR: track 0.00 -> 20.4 mm
- net VOUTL: track 25.3 -> 40.9 mm, vias 2 -> 0
- net N$34: track 15.6 -> 0.00 mm
- net +3V3: track 31.0 -> 17.2 mm, vias 5 -> 6
- net /JACKSENSE: track 13.2 -> 0.00 mm
- net N$29: track 12.3 -> 0.00 mm
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- added copper zone on layer 15, net +5V
Other:
- board size 32.8 x 56.9 mm -> 32.8 x 54.3 mm
- board text added: "SPH0645LM4H UDA1334A MAX98306 PCF8574 v0.13 - 07/19 Adam Keher"
- board text removed: "-6dB"
- board text removed: "0dB"
- board text removed: "3dB"
- board text removed: "6dB"
- board text removed: "BUTTONS"
- board text removed: "G0"
- board text removed: "G1"
- board text removed: "HPGAIN"
- board text removed: "SPH0645LM4H UDA1334A MAX98306 PCF8574 v0.20 - 08/19 Adam Keher"
