File: eagle/Pico Audio v0.20.brd (EAGLE design)
At the start: 32.8 x 54.3 mm, 72 parts, among them IC1 MIC_I2S_SPH0645, J1 OUTR, J2 OUTL, J3 GPIO Expander Pins, J4 TinyPICO, J5 TinyPICO, J6 Pin Out 2, J8 Pin Out 1, U1 UDA1334ATS, U2 MAX98306ETD+T, U3 PCF8574, U4 NCP170AMX300TCG, X1 STEREOJACKSTX3120-5B

Commit message: v0.20 Update
Parts:
- removed AK74LOGO2: AK74_LOGOAK74_LOGO_SMALL, AK74:AK74_LOGO_MEDIUM
- removed J8: Pin Out 1, SparkFun-Connectors:1X08_NO_SILK
- added AK74LOGO1: AK74_LOGOAK74_LOGO_SMALL, AK74:AK74_LOGO_MEDIUM
- added C22, C23, C24, C25, C26, C27, C28: 1uF, rcl:C0402K
- added C29, C31: 0.1uF, rcl:C0402K
- added C30: 10uF, rcl:C0603K
- added J7: Pin Out 2, SparkFun-Connectors:1X07_NO_SILK
- added JP2: SPKGAIN, pinhead:2X04
- added R23: 100K, rcl:R0402
- added R24: 10K, rcl:R0402
- added R25, R26: 270, rcl:R0402
- added R27, R28: 4.7K, rcl:R0402
- added S4, S5: SKSCLDE010, AK74:SKSCLDE010
- added U5: MAX98306ETD+T, microbuilder:TDFN14_3X3MM
- added U6: PCF8574, AK74:QFN-16-3MM
- C11: value 10uF -> 0.1uF; device rcl:C0603K -> rcl:C0402K
- C12: value 0.1uF -> 10uF; device rcl:C0402K -> rcl:C0603K
- C15, C5: value 1uF -> 10uF; device rcl:C0402K -> rcl:C0603K
- C16: value 1uF -> 2.2uF
- C17, C3: value 10uF -> 1uF; device rcl:C0603K -> rcl:C0402K
- C18: value 0.1uF -> 1uF
- C19: value 0.1uF -> 2.2uF
- C4: value 0.1uF -> 220pf
- C6: value 220pf -> 0.1uF
- J1: value OUTR -> TinyPICO; device microbuilder:TERMBLOCK_1X2-3.5MM -> UnexpectedMaker:1X10_NO_SILK
- J2: value OUTL -> TinyPICO; device microbuilder:TERMBLOCK_1X2-3.5MM -> UnexpectedMaker:1X10_NO_SILK
- J3: value GPIO Expander Pins -> Pin Out 1
- J4: value TinyPICO -> GPIO Expander Pins; device UnexpectedMaker:1X10_NO_SILK -> SparkFun-Connectors:1X08_NO_SILK
- J5: value TinyPICO -> OUTR; device UnexpectedMaker:1X10_NO_SILK -> microbuilder:TERMBLOCK_1X2-3.5MM
- J6: value Pin Out 2 -> OUTL; device SparkFun-Connectors:1X07_NO_SILK -> microbuilder:TERMBLOCK_1X2-3.5MM
- JP1: value GAIN -> HPGAIN; device pinhead:2X04 -> pinhead:2X02
- R10: value 100 -> 10K
- R11: value 100 -> 220K
- R12: value 10K -> 220K
- R13: value 10K -> 100
- R14: value 270 -> 100
- R16: value 100K -> 270
- R17: value 100K -> 10K
- R19: value 10K -> 100K
- R20: value 4.7K -> 49.9K
- R21: value 4.7K -> 270
- R22: value 270 -> 100K
- R6: value 10K -> 68
- R8: value 68 -> 10K
- S1, S2, S3: value MOMENTARY-SWITCH-SPST-SMD-4.6X2.8MM -> SKSCLDE010; device SparkFun-Switches:TACTILE_SWITCH_SMD_4.6X2.8MM -> AK74:SKSCLDE010
- U2: value MAX98306ETD+T -> TPA6132A2RTER; device microbuilder:TDFN14_3X3MM -> TPA6132A2RTER:QFN50P300X300X80-16N
- U3: value PCF8574 -> NCP170AMX300TCG; device AK74:QFN-16-3MM -> NCP170AMX300TCG:VREG_NCP170AMX300TCG
- U4: value NCP170AMX300TCG -> NC7SZ04; device NCP170AMX300TCG:VREG_NCP170AMX300TCG -> AK74:MICROPAK-6
- moved MH3 51.6 mm to (2.54, 53.7)
- moved MH2 49.1 mm to (2.54, 2.06)
- moved JP1 48.5 mm to (15.3, 50.5), turned to 0 degrees
- moved R17 32.2 mm to (22.1, 38.9), turned to 180 degrees
- moved R14 25.7 mm to (3.33, 22.2), turned to 0 degrees
- moved R21 24.7 mm to (29.1, 22.5), turned to 180 degrees
- moved R22 24.4 mm to (8.57, 8.57), turned to 0 degrees
- moved R20 23.8 mm to (31.9, 37.6), turned to 270 degrees
- moved J4 22.6 mm to (19.2, 46.7), turned to 180 degrees
- moved R16 22.3 mm to (29.1, 17.5), turned to 180 degrees
- moved J5 21.4 mm to (3.81, 38.7), turned to 270 degrees
- moved C12 21.4 mm to (7.30, 30.2)
- moved U4 20.4 mm to (31.0, 33.7), turned to 270 degrees
- moved C10 20.1 mm to (15.2, 11.7)
- moved J3 18.0 mm to (1.37, 44.1), turned to 0 degrees
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- renumbered PWR to LED2, SDCRD to LED1
Connections:
- removed net SHUTDOWN: R15.2, U2.P$2
- removed net VINL: C15.2, R18.2, X1.4
- removed net VINR: C16.2, R19.2, X1.3
- new net /JACKSENSE: R24.2, U4.4, U5.P$2
- new net G0: JP1.2, U2.6
- new net G1: JP1.4, U2.7
- new net JACKSENSE: C24.1, R20.2, U4.2
- new net N$12: C18.2, U2.4
- new net N$13: R17.1, U2.13
- new net N$23: C19.1, U2.12
- new net N$29: R18.1, U2.5, X1.2
- new net N$30: U2.16, X1.5
- new net N$31: C21.2, U2.11
- new net N$32: C21.1, U2.9
- new net N$33: C22.1, U2.8
- new net N$34: R19.2, R20.1, X1.3
- new net N$6: C26.1, U5.P$4
- new net N$7: C28.1, U5.P$6
- new net N$9: C17.2, U2.1
- net +3V3: now also C10.1, C3.1, C4.1, J1.4, J3.1, R15.2; no longer C12.1, C5.1, C6.1, J4.4, J8.1, R13.2
- net +3V3#2: now also C15.1, C16.1, C23.1, C29.1, JP1.1, JP1.3, R17.2, R19.1, R27.2, R28.2, U2.14, U4.6, U6.1; no longer C19.1, C21.1, R20.2, R21.2, U4.1
- net +5V: now also C30.1, C31.1, J1.3, J3.2, JP2.3, R23.2, U3.3, U3.4, U5.P$11, U5.P$12; no longer C17.1, C18.1, J4.3, J8.2, JP1.3, R15.1, R17.2, U2.P$11, U2.P$12, U4.3, U4.4
- net AGND: now also C12.2, C26.2, C28.2, C5.2, C6.2, R11.2, R12.2, R25.1, R26.1, U2.15; no longer C10.2, C3.2, C4.2, R18.1, R19.1, U2.P$4, U2.P$6
- net DAC_BCK: now also J1.9; no longer J4.9
- net DAC_DIN: now also J2.5; no longer J5.5
- net DAC_WS: now also J1.10; no longer J4.10
- net DEEM: now also J3.4; no longer J8.4
- net GAIN1: now also JP2.2, JP2.4, JP2.6, JP2.8, U5.P$5; no longer JP1.2, JP1.4, JP1.6, JP1.8, U2.P$5
- net GND: now also C10.2, C15.2, C16.2, C22.2, C23.2, C24.2, C29.2, C3.2, C30.2, C31.2, C4.2, J1.2, J2.10, J3.3, JP2.7, R10.1, R18.2, R21.1, R24.1, R8.1, S4.3, S4.4, S5.3, S5.4, U2.10, U2.17, U2.2, U2.3, U3.5, U4.3, U5.P$1, U5.P$8, U5.P$THERMAL, U6.2, U6.3, U6.4, U6.9, U6.P$1; no longer C12.2, C17.2, C18.2, C21.2, C5.2, C6.2, J4.2, J5.10, J8.3, JP1.7, R12.1, R16.1, R6.1, U2.P$1, U2.P$8, U2.P$THERMAL, U3.3, U3.4, U3.9, U3.P$1, U4.2, U4.5
- net GPIO21: now also J2.6, J7.4; no longer J5.6, J6.4
- net GPIO27: now also J1.8, J7.5; no longer J4.8, J6.5
- net MIC_BCK: now also J1.6, J3.7; no longer J4.6, J8.7
- net MIC_DOUT: now also J1.7, J3.5, R6.1; no longer J4.7, J8.5, R8.1
- net MIC_WS: now also J1.5, J3.6; no longer J4.5, J8.6
- net MISO: now also J2.2, J7.2, R10.2; no longer J5.2, J6.2, R12.2
- net MOSI: now also J2.1, J7.1; no longer J5.1, J6.1
- net MUTE: now also J3.8; no longer J8.8
- net N$1: now also C5.1, C6.1; no longer C3.1, C4.1
- net N$10: now also R7.2; no longer R6.2
- net N$11: now also R8.2; no longer R7.2
- net N$14: now also C12.1; no longer C10.1
- net N$16: now also R12.1, R14.2; no longer R11.2
- net N$17: now also J6.2, U5.P$9; no longer J2.2, U2.P$9
- net N$18: now also J5.2, U5.P$14; no longer J1.2, U2.P$14
- net N$19: now also R11.1, R13.2; no longer R10.2
- net N$2: now also C25.1, U5.P$3; no longer C15.1, U2.P$3
- net N$20: now also R1.2; no longer R2.2
- net N$22: now also R6.2; no longer R8.2
- net N$24: now also JP2.1, R23.1; no longer JP1.1, R17.1
- net N$25: now also JP2.5, R22.2; no longer JP1.5, R16.2
- net N$26: now also J5.1, U5.P$13; no longer J1.1, U2.P$13
- net N$27: now also R16.2; no longer R14.2
- net N$28: now also J6.1, U5.P$10; no longer J2.1, U2.P$10
- net N$3: now also R2.2; no longer R1.2
- net N$4: now also C27.1, U5.P$7; no longer C16.1, U2.P$7
- net N$8: now also R21.2; no longer R22.2
- net P0: now also J4.1, U6.5; no longer J3.1, U3.5
- net P1: now also J4.2, U6.6; no longer J3.2, U3.6
- net P2: now also J4.3, U6.7; no longer J3.3, U3.7
- net P3: now also J4.4, S1.1, S1.2, U6.8; no longer J3.4, U3.8
- net P4: now also J4.5, S2.1, S2.2, U6.10; no longer J3.5, U3.10
- net P5: now also J4.6, S3.1, S3.2, U6.11; no longer J3.6, S1.1, S1.2, U3.11
- net P6: now also J4.7, S4.1, S4.2, U6.12; no longer J3.7, S2.1, S2.2, U3.12
- net P7: now also J4.8, S5.1, S5.2, U6.13; no longer J3.8, S3.1, S3.2, U3.13
- net RESET: now also J2.9; no longer J5.9
- net SCK: now also J2.3, J7.3; no longer J5.3, J6.3
- net SCL: now also J2.8, J7.7, R27.1, U6.15; no longer J5.8, J6.7, R20.1, U3.15
- net SDA: now also J2.7, J7.6, R28.1, U6.16; no longer J5.7, J6.6, R21.1, U3.16
- net SD_CS: now also J2.4, R15.1, R16.1; no longer J5.4, R13.1, R14.1
- net VBAT: now also J1.1; no longer J4.1
- net VOUTL: now also C17.1, C25.2, R13.1, R26.2; no longer R10.1, X1.5
- net VOUTR: now also C18.1, C27.2, R14.1, R25.2; no longer R11.1, X1.2
Routing:
- net +5V: track 10.4 -> 85.1 mm, vias 4 -> 3
- net P3: track 6.75 -> 39.7 mm
- net GND: track 54.7 -> 81.1 mm, vias 28 -> 34
- net G0: track 0.00 -> 26.2 mm, vias 0 -> 1
- net P4: track 6.51 -> 30.6 mm
- net G1: track 0.00 -> 23.9 mm, vias 0 -> 1
- net N$30: track 0.00 -> 23.7 mm
- net VINL: track 22.7 -> 0.00 mm
- net +3V3#2: track 16.2 -> 38.9 mm, vias 6 -> 10
- net VINR: track 20.4 -> 0.00 mm
- net VOUTL: track 40.9 -> 25.3 mm, vias 0 -> 2
- net N$34: track 0.00 -> 15.6 mm
- net +3V3: track 17.2 -> 31.0 mm, vias 6 -> 5
- net /JACKSENSE: track 0.00 -> 13.2 mm
- net N$29: track 0.00 -> 12.3 mm
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- removed copper zone on layer 15, net +5V
Other:
- board size 32.8 x 54.3 mm -> 32.8 x 56.9 mm
- board text added: "-6dB"
- board text added: "0dB"
- board text added: "3dB"
- board text added: "6dB"
- board text added: "BUTTONS"
- board text added: "G0"
- board text added: "G1"
- board text added: "HPGAIN"
- board text added: "SPH0645LM4H UDA1334A MAX98306 PCF8574 v0.20 - 08/19 Adam Keher"
- board text removed: "SPH0645LM4H UDA1334A MAX98306 PCF8574 v0.13 - 07/19 Adam Keher"
