File: eagle/Pico Audio v0.20.sch (EAGLE design)
At the start: 71 parts, among them IC1 MIC_I2S_SPH0645, J1 OUTR, J2 OUTL, J3 GPIO Expander Pins, J4 TinyPICO, J5 TinyPICO, J6 Pin Out 2, J8 Pin Out 1, U1 UDA1334ATS, U2 MAX98306ETD+T, U3 PCF8574, U4 NCP170AMX300TCG, X1 STEREOJACKSTX3120-5B

Commit message: v0.20 Update
Parts:
- removed AK74LOGO2: AK74_LOGOAK74_LOGO_SMALL, AK74:AK74_LOGOAK74_LOGO_SMALL
- removed J8: Pin Out 1, SparkFun-Connectors:CONN_08NO_SILK_FEMALE_PTH
- removed PWR: GREEN, led:LEDCHIP-LED0805
- removed SDCRD: RED, led:LEDCHIP-LED0805
- added AK74LOGO1: AK74_LOGOAK74_LOGO_SMALL, AK74:AK74_LOGOAK74_LOGO_SMALL
- added C22, C23, C24, C25, C26, C27, C28: 1uF, rcl:C-USC0402K
- added C29, C31: 0.1uF, rcl:C-USC0402K
- added C30: 10uF, rcl:C-USC0603K
- added J7: Pin Out 2, SparkFun-Connectors:CONN_07NO_SILK
- added JP2: SPKGAIN, pinhead:PINHD-2X4
- added LED1: RED, led:LEDCHIP-LED0805
- added LED2: GREEN, led:LEDCHIP-LED0805
- added R23: 100K, rcl:R-US_R0402
- added R24: 10K, rcl:R-US_R0402
- added R25, R26: 270, rcl:R-US_R0402
- added R27, R28: 4.7K, rcl:R-US_R0402
- added S4, S5: SKSCLDE010, AK74:SKSCLDE010
- added U5: MAX98306ETD+T, microbuilder:AUDIOAMP_MAX98306
- added U6: PCF8574, AK74:PCF8574
- C11: value 10uF -> 0.1uF; device rcl:C-USC0603K -> rcl:C-USC0402K
- C12: value 0.1uF -> 10uF; device rcl:C-USC0402K -> rcl:C-USC0603K
- C15, C5: value 1uF -> 10uF; device rcl:C-USC0402K -> rcl:C-USC0603K
- C16: value 1uF -> 2.2uF
- C17, C3: value 10uF -> 1uF; device rcl:C-USC0603K -> rcl:C-USC0402K
- C18: value 0.1uF -> 1uF
- C19: value 0.1uF -> 2.2uF
- C4: value 0.1uF -> 220pf
- C6: value 220pf -> 0.1uF
- J1: value OUTR -> TinyPICO; device microbuilder:TERMBLOCK_1X2 -> UnexpectedMaker:TINYPICO_HEADER_10NO_SILK_PTH_FEMALE
- J2: value OUTL -> TinyPICO; device microbuilder:TERMBLOCK_1X2 -> UnexpectedMaker:TINYPICO_HEADER_10NO_SILK_PTH_FEMALE
- J3: value GPIO Expander Pins -> Pin Out 1
- J4: value TinyPICO -> GPIO Expander Pins; device UnexpectedMaker:TINYPICO_HEADER_10NO_SILK_PTH_FEMALE -> SparkFun-Connectors:CONN_08NO_SILK_FEMALE_PTH
- J5: value TinyPICO -> OUTR; device UnexpectedMaker:TINYPICO_HEADER_10NO_SILK_PTH_FEMALE -> microbuilder:TERMBLOCK_1X2
- J6: value Pin Out 2 -> OUTL; device SparkFun-Connectors:CONN_07NO_SILK -> microbuilder:TERMBLOCK_1X2
- JP1: value GAIN -> HPGAIN; device pinhead:PINHD-2X4 -> pinhead:PINHD-2X2
- R10: value 100 -> 10K
- R11: value 100 -> 220K
- R12: value 10K -> 220K
- R13: value 10K -> 100
- R14: value 270 -> 100
- R16: value 100K -> 270
- R17: value 100K -> 10K
- R19: value 10K -> 100K
- R20: value 4.7K -> 49.9K
- R21: value 4.7K -> 270
- R22: value 270 -> 100K
- R6: value 10K -> 68
- R8: value 68 -> 10K
- S1, S2, S3: value MOMENTARY-SWITCH-SPST-SMD-4.6X2.8MM -> SKSCLDE010; device SparkFun-Switches:MOMENTARY-SWITCH-SPST-SMD-4.6X2.8MM -> AK74:SKSCLDE010
- U2: value MAX98306ETD+T -> TPA6132A2RTER; device microbuilder:AUDIOAMP_MAX98306 -> TPA6132A2RTER:TPA6132A2RTER
- U3: value PCF8574 -> NCP170AMX300TCG; device AK74:PCF8574 -> NCP170AMX300TCG:NCP170AMX300TCG
- U4: value NCP170AMX300TCG -> NC7SZ04; device NCP170AMX300TCG:NCP170AMX300TCG -> AK74:NC7SZ04
Connections:
- removed net SHUTDOWN: R15.2, U2.SHDN
- removed net VINL: C15.2, R18.2, X1.4
- removed net VINR: C16.2, R19.2, X1.3
- new net /JACKSENSE: R24.2, U4.Y, U5.SHDN
- new net G0: JP1.2, U2.G0
- new net G1: JP1.4, U2.G1
- new net JACKSENSE: C24.1, R20.2, U4.A
- new net N$12: C18.2, U2.INR-
- new net N$13: R17.1, U2.EN
- new net N$23: C19.1, U2.HPVDD
- new net N$29: R18.1, U2.OUTR, X1.2
- new net N$30: U2.OUTL, X1.5
- new net N$31: C21.2, U2.CPP
- new net N$32: C21.1, U2.CPN
- new net N$33: C22.1, U2.HPVSS
- new net N$34: R19.2, R20.1, X1.3
- new net N$6: C26.1, U5.INL-
- new net N$7: C28.1, U5.INR-
- new net N$9: C17.2, U2.INL-
- net +3V3: now also C10.1, C3.1, C4.1, J1.4, J3.1, LED2.A, R15.2; no longer C12.1, C5.1, C6.1, J4.4, J8.1, PWR.A, R13.2
- net +3V3#2: now also C15.1, C16.1, C23.1, C29.1, JP1.1, JP1.3, R17.2, R19.1, R27.2, R28.2, U2.VDD, U3.OUT, U4.VCC, U6.VCC; no longer C19.1, C21.1, R20.2, R21.2, U3.VCC, U4.OUT
- net +5V: now also C30.1, C31.1, J1.3, J3.2, JP2.3, R23.2, U3.EN, U3.IN, U5.PVDD@1, U5.PVDD@2; no longer C17.1, C18.1, J4.3, J8.2, JP1.3, R15.1, R17.2, U2.PVDD@1, U2.PVDD@2, U4.EN, U4.IN
- net AGND: now also C12.2, C26.2, C28.2, C5.2, C6.2, R11.2, R12.2, R25.1, R26.1, U2.SGND; no longer C10.2, C3.2, C4.2, R18.1, R19.1, U2.INL-, U2.INR-
- net DAC_BCK: now also J1.9; no longer J4.9
- net DAC_DIN: now also J2.5; no longer J5.5
- net DAC_WS: now also J1.10; no longer J4.10
- net DEEM: now also J3.4; no longer J8.4
- net GAIN1: now also JP2.2, JP2.4, JP2.6, JP2.8, U5.GAIN; no longer JP1.2, JP1.4, JP1.6, JP1.8, U2.GAIN
- net GND: now also C10.2, C15.2, C16.2, C22.2, C23.2, C24.2, C29.2, C3.2, C30.2, C31.2, C4.2, J1.2, J2.10, J3.3, JP2.7, R10.1, R18.2, R21.1, R24.1, R8.1, S4.2, S5.2, U2.EP, U2.INL+, U2.INR+, U2.PGND, U3.EXP, U5.PGND@1, U5.PGND@2, U5.THERMAL, U6.A0, U6.A1, U6.A2, U6.GND; no longer C12.2, C17.2, C18.2, C21.2, C5.2, C6.2, J4.2, J5.10, J8.3, JP1.7, R12.1, R16.1, R6.1, U2.PGND@1, U2.PGND@2, U2.THERMAL, U3.A0, U3.A1, U3.A2, U4.EXP
- net GPIO21: now also J2.6, J7.4; no longer J5.6, J6.4
- net GPIO27: now also J1.8, J7.5; no longer J4.8, J6.5
- net MIC_BCK: now also J1.6, J3.7; no longer J4.6, J8.7
- net MIC_DOUT: now also J1.7, J3.5, R6.1; no longer J4.7, J8.5, R8.1
- net MIC_WS: now also J1.5, J3.6; no longer J4.5, J8.6
- net MISO: now also J2.2, J7.2, R10.2; no longer J5.2, J6.2, R12.2
- net MOSI: now also J2.1, J7.1; no longer J5.1, J6.1
- net MUTE: now also J3.8; no longer J8.8
- net N$1: now also C5.1, C6.1; no longer C3.1, C4.1
- net N$10: now also R7.2; no longer R6.2
- net N$11: now also R8.2; no longer R7.2
- net N$14: now also C12.1; no longer C10.1
- net N$16: now also R12.1, R14.2; no longer R11.2
- net N$17: now also J6.2, U5.OUTR-; no longer J2.2, U2.OUTR-
- net N$18: now also J5.2, U5.OUTL-; no longer J1.2, U2.OUTL-
- net N$19: now also R11.1, R13.2; no longer R10.2
- net N$2: now also C25.1, U5.INL+; no longer C15.1, U2.INL+
- net N$20: now also R1.2; no longer R2.2
- net N$22: now also R6.2; no longer R8.2
- net N$24: now also JP2.1, R23.1; no longer JP1.1, R17.1
- net N$25: now also JP2.5, R22.2; no longer JP1.5, R16.2
- net N$26: now also J5.1, U5.OUTL+; no longer J1.1, U2.OUTL+
- net N$27: now also LED1.C, R16.2; no longer R14.2, SDCRD.C
- net N$28: now also J6.1, U5.OUTR+; no longer J2.1, U2.OUTR+
- net N$3: now also R2.2; no longer R1.2
- net N$4: now also C27.1, U5.INR+; no longer C16.1, U2.INR+
- net N$8: now also LED2.C, R21.2; no longer PWR.C, R22.2
- net P0: now also J4.1, U6.P0; no longer J3.1, U3.P0
- net P1: now also J4.2, U6.P1; no longer J3.2, U3.P1
- net P2: now also J4.3, U6.P2; no longer J3.3, U3.P2
- net P3: now also J4.4, S1.1, U6.P3; no longer J3.4, U3.P3
- net P4: now also J4.5, S2.1, U6.P4; no longer J3.5, U3.P4
- net P5: now also J4.6, S3.1, U6.P5; no longer J3.6, S1.1, U3.P5
- net P6: now also J4.7, S4.1, U6.P6; no longer J3.7, S2.1, U3.P6
- net P7: now also J4.8, S5.1, U6.P7; no longer J3.8, S3.1, U3.P7
- net RESET: now also J2.9; no longer J5.9
- net SCK: now also J2.3, J7.3, LED1.A; no longer J5.3, J6.3, SDCRD.A
- net SCL: now also J2.8, J7.7, R27.1, U6.SCL; no longer J5.8, J6.7, R20.1, U3.SCL
- net SDA: now also J2.7, J7.6, R28.1, U6.SDA; no longer J5.7, J6.6, R21.1, U3.SDA
- net SD_CS: now also J2.4, R15.1, R16.1; no longer J5.4, R13.1, R14.1
- net VBAT: now also J1.1; no longer J4.1
- net VOUTL: now also C17.1, C25.2, R13.1, R26.2; no longer R10.1, X1.5
- net VOUTR: now also C18.1, C27.2, R14.1, R25.2; no longer R11.1, X1.2
Other:
- note added: "* CHECK LED POLARITY AND TEST PULLDOWNS W/ LCD & SDCARD"
- note added: "* CHECK LEFT & RIGHT ROUTING AT ALL STAGES AND CHECK HEADPHONE PINS"
- note added: "G0|G1 |DB --+---+---- - | - |-6dB x | - | 0db - | x | 3db x | x | 6db"
- moved on the sheet: C1, C10, C11, C12, C13, C14, C15, C16, C17, C18, C19, C2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
